Commit message: slam_project init

File: urdf/_d435.urdf.xacro (robot description, xacro)
@@ -40,5 +40,5 @@
         <geometry>
           <!-- <box size="${d435_cam_width} ${d435_cam_height} ${d435_cam_depth}"/> -->
-	  <mesh filename="package://racer_bot/meshes/d435.dae" />
+	  <mesh filename="package://slam_project/meshes/d435.dae" />
           <!--<mesh filename="package://realsense2_camera/meshes/d435/d435.dae" />-->
         </geometry>

File: urdf/racer_bot.xacro (robot description, xacro)
@@ -1,6 +1,6 @@
 <?xml version="1.0"?>
-<robot name="racer_bot" xmlns:xacro="http://www.ros.org/wiki/xacro">
-    <xacro:include filename="$(find racer_bot)/urdf/material.xacro" />
-    <xacro:include filename="$(find racer_bot)/urdf/robot.gazebo" />
-    <xacro:include filename="$(find racer_bot)/urdf/robot.xacro" />
+<robot name="slam_project" xmlns:xacro="http://www.ros.org/wiki/xacro">
+    <xacro:include filename="$(find slam_project)/urdf/material.xacro" />
+    <xacro:include filename="$(find slam_project)/urdf/robot.gazebo" />
+    <xacro:include filename="$(find slam_project)/urdf/robot.xacro" />
 </robot>

File: urdf/realsense-RS200.macro.xacro (robot description, xacro)
@@ -20,5 +20,5 @@
             <origin rpy="${3*pi/2} 0 ${3*pi/2}" xyz="0.01 0 0"/>
             <geometry>
-                <mesh filename="package://racer_bot/meshes/d435.dae"/>
+                <mesh filename="package://slam_project/meshes/d435.dae"/>
             </geometry>
         </visual>

File: urdf/robot.xacro (robot description, xacro)
@@ -1,5 +1,5 @@
 <?xml version='1.0'?>
-<robot name="racer_bot" xmlns:xacro="http://www.ros.org/wiki/xacro">
-  <xacro:include filename="$(find racer_bot)/urdf/realsense-RS200.macro.xacro"/>
+<robot name="slam_project" xmlns:xacro="http://www.ros.org/wiki/xacro">
+  <xacro:include filename="$(find slam_project)/urdf/realsense-RS200.macro.xacro"/>
   <link name="robot_footprint"></link>
   <joint name="robot_footprint_joint" type="fixed">
@@ -109,5 +109,5 @@
 			<origin xyz="0 0 0" rpy="0 0 0"/>
 			<geometry>
-				<mesh filename="package://racer_bot/meshes/hokuyo.dae"/>
+				<mesh filename="package://slam_project/meshes/hokuyo.dae"/>
 			</geometry>
 		</visual>
