Commit message: SLAM works
build from source pakage error.
spends a lot of mem space due to the scan from d435

File: urdf/robot.xacro (robot description, xacro)
@@ -97,9 +97,38 @@
   <xacro:wheel prefix="right" reflect="-1" />
   <xacro:wheel prefix="left" reflect="1" />
+  <link name="camera_support_link">
+		<visual name="camera_support_visual">
+			<origin xyz="0 0 0" rpy="0 0 0"/>
+			<geometry>
+				<box size=".05 .05 .8"/>
+			</geometry>
+		</visual>
+		<collision name="camera_support_collision">
+			<origin xyz="0 0 0" rpy="0 0 0"/>
+			<geometry>
+				<box size="0.05 0.05 0.8"/>
+			</geometry>
+		</collision>
+		<inertial>
+        <mass value="0.1"/>
+        <origin xyz="0 0 0" rpy="0 0 0"/>
+        <inertia
+                ixx="1e-6" ixy="0" ixz="0"
+                iyy="1e-6" iyz="0"
+                izz="1e-6"
+        />
+    </inertial>
+	</link>
     <!-- Create camera instance -->
     <xacro:realsense-rs200/>
+  <joint name="camera_support_joint" type="fixed">
+    <origin xyz="0.0 0.0 0.4" rpy="0.0 0.0 0.0"/>
+    <parent link="chassis"/>
+    <child link="camera_support_link"/>
+    <limit effort="1000" velocity="100"/>
+  </joint>
   <joint name="camera_joint" type="fixed">
-    <origin xyz="0.2 0.0 0.0" rpy="0.0 0.0 0.0"/>
-    <parent link="chassis"/>
+    <origin xyz="0.0 0.0 0.42" rpy="0.0 0.0 0.0"/>
+    <parent link="camera_support_link"/>
     <child link="rs200_camera"/>
     <limit effort="1000" velocity="100"/>
